File: pcb/PowerPod/current.kicad_sch (KiCad schematic)
At the start: 4 parts, among them IC3 CC6904SO-10A

Commit message: finished layout
Parts:
- added Q1: DMP3017SFG-7, DMP3007SFG7, symbol Transistor_JLC:DMP3017SFG-7
- added Q2: DTC143ECA-TP, SOT95P237X125-3N, symbol Transistor_JLC:DTC143ECA-TP
- added R19: 1k, Resistor_SMD:R_0402_1005Metric, symbol Resistor_JLC:1k
- added R20: 10k, Resistor_SMD:R_0402_1005Metric, symbol Resistor_JLC:10k
- added R21: DNF_0805, Resistor_SMD:R_0805_2012Metric_Pad1.20x1.40mm_HandSolder, symbol personal:DNF_0805
- added TP5 (x2): TestPoint, TestPoint:TestPoint_Pad_D1.0mm, symbol Connector:TestPoint
Connections:
- net GND: now also Q2.2
- net VIN: now also Q1.1, Q1.2, Q1.3, R20.1, R21.1; no longer IC3.1 (IP+), IC3.2 (IP+)
- net V_CURRENT: now also TP5.1
- new net: Q1.4 (G), R19.1, R20.2
- new net: IC3.1 (IP+), IC3.2 (IP+), Q1.5 (D_1), Q1.6, Q1.7, Q1.8, Q1.9, R21.2, TP5.1
- new net: Q2.3, R19.2
- new net OUTPUT_EN: Q2.1
Other:
- note added: "HIGH -> Off LOW -> On"
- note added: "IN"
- note added: "OUT"
- note added: "Output Enable"
