File: pcb/PowerPod/power.kicad_sch (KiCad schematic)
At the start: 15 parts, among them IC4 TPS62175DQCT

Commit message: finished layout
Parts:
- added TP5 (x5): TestPoint, TestPoint:TestPoint_Pad_D1.0mm, symbol Connector:TestPoint
Connections:
- net 3V3: now also R4.2, TP5.1; no longer C2.1, C3.1, IC4.10 (VOS), L1.2, R1.1, R2.1, R5.2
- net GND: now also TP5.1, TP5.1, TP5.1; no longer R4.2
- net VIN: now also TP5.1
- net at R4.1: now also C2.1, C3.1, IC4.10 (VOS), L1.2, R1.1, R2.1, R5.2; no longer IC4.4 (NC)
