File: pcb/PowerPod/PowerPod.kicad_sch (KiCad schematic)
At the start: 3 parts, among them J3 KF350-3.5-2P

Commit message: finished layout
Parts:
- added H1, H2, H3, H4: MountingHole, MountingHole:MountingHole_2.2mm_M2, symbol Mechanical:MountingHole
- added TP5: TestPoint, TestPoint:TestPoint_Pad_D1.0mm, symbol Connector:TestPoint
Connections:
- net Current Sensor + Output Control/VOUT: now also TP5.1
Other:
- sheet Current Sensor renamed Current Sensor + Output Control
- sheet Current Sensor + Output Control ports: added OUTPUT_EN; removed none
- sheet Microcontroller ports: added OUTPUT_EN; removed none
- moved on the sheet: C21, J3
