File: pcb/PowerPod/mcu.kicad_sch (KiCad schematic)
At the start: 30 parts, among them IC5 ESP32-C3FH4, J2 TC2050-IDC, J5 Conn_01x06, Y2 SX25Y040000BF1T-C

Commit message: finished layout
Parts:
- added TP1, TP2, TP6: TestPoint, TestPoint:TestPoint_Pad_D1.0mm, symbol Connector:TestPoint
Connections:
- net EN: now also TP6.1
- net GPIO0: now also J5.3 (Pin_3); no longer J5.4 (Pin_4)
- net GPIO1: now also J5.2 (Pin_2); no longer J5.5 (Pin_5)
- net SCL: now also TP2.1
- net SDA: now also TP1.1
- net U0RXD: now also J5.4 (Pin_4); no longer J5.2 (Pin_2)
- net U0TXD: now also J5.5 (Pin_5); no longer J5.3 (Pin_3)
- net GPIO3 renamed OUTPUT_EN
Other:
- moved on the sheet: R12

Commit message: changed gpio pins
Parts:
- removed R13, R14: 10k, Resistor_SMD:R_0402_1005Metric, symbol Resistor_JLC:10k
- removed TP1, TP2: TestPoint, TestPoint:TestPoint_Pad_D1.0mm, symbol Connector:TestPoint
Connections:
- net SCL: now also IC5.4 (XTAL_32K_P); no longer IC5.15 (GPIO9), S2.1
- net SDA: now also IC5.5 (XTAL_32K_N); no longer IC5.14 (GPIO8)
- net GPIO0 renamed GPIO9
- net GPIO9: now also IC5.15 (GPIO9), S2.1; no longer IC5.4 (XTAL_32K_P)
- net GPIO1 renamed GPIO8
- net GPIO8: now also IC5.14 (GPIO8); no longer IC5.5 (XTAL_32K_N)
