File: pcb/Spark-Analyzer/mcu.kicad_sch (KiCad schematic)
At the start: 29 parts, among them IC5 ESP32-C3FH4, J2 TC2050-IDC, J5 Conn_01x06, Y2 SX25Y040000BF1T-C

Commit message: First app release and updated PCBA
Parts:
- removed AE1: ANT3216LL00R2400A, Resistor_SMD:R_1206_3216Metric_Pad1.30x1.75mm_HandSolder, symbol RF_JLC:ANT3216LL00R2400A
- removed D1: Green_0603, LED_SMD:LED_0603_1608Metric, symbol Diode_JLC:Green_0603
- removed R10: 0, Resistor_SMD:R_0805_2012Metric_Pad1.20x1.40mm_HandSolder, symbol Resistor_JLC:0
- removed R15: DNF_0402, Resistor_SMD:R_0402_1005Metric, symbol personal:DNF_0402
- removed TP6: TestPoint, TestPoint:TestPoint_Pad_D1.0mm, symbol Connector:TestPoint
- added D3: Yellow_0603, LED_SMD:LED_0603_1608Metric, symbol Diode_JLC:Yellow_0603
- added D4: Green_0603, LED_SMD:LED_0603_1608Metric, symbol Diode_JLC:Green_0603
- added R16: 2.7k, Resistor_SMD:R_0402_1005Metric, symbol Resistor_JLC:2.7k
Connections:
- net GND: now also R16.2
- net GPIO8: now also D4.2 (A)
- net OUTPUT_EN: now also D3.2 (A)
- net at R16.1: now also D3.1 (K)
- net at C10.1, L2.1: now also AE2.1 (A)
- new net: D4.1 (K), R16.1
- no-connect marks 8 -> 7
Other:
- note added: "OUTPUT LED"
- note removed: "BLINK"
- moved on the sheet: R16

Commit message: Added silkscreen symbols and texts
Other:
- note added: "DEBUG LED"
Changed lines of the file:
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@@
     (effects (font (size 2.54 2.54) (thickness 0.508) bold) (justify left bottom))
   )
-  (text "OUTPUT LED" (at 347.98 182.88 0)
+  (text "DEBUG LED" (at 347.98 182.88 0)
     (effects (font (size 2.54 2.54) (thickness 0.508) bold) (justify left bottom))
   )

Commit message: Wired sensor and changed connector
Parts:
- removed J2: TC2050-IDC, TC2050-IDC, symbol personal:TC2050-IDC
- removed R11, R9: 0, Resistor_SMD:R_0805_2012Metric_Pad1.20x1.40mm_HandSolder, symbol Resistor_JLC:0
Connections:
- no-connect marks 7 -> 6
Other:
- note removed: "JTAG"
Changed lines of the file:
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@@
   (junction (at 163.83 81.915) (diameter 0) (color 0 0 0 0)
-  )
-  (junction (at 100.33 196.85) (diameter 0) (color 0 0 0 0)
   )
   (junction (at 142.24 159.385) (diameter 0) (color 0 0 0 0)
@@
   (no_connect (at 222.885 134.62))
   (no_connect (at 222.885 144.78))
-  (no_connect (at 87.63 176.53))
   (no_connect (at 222.885 142.24))
   (no_connect (at 222.885 139.7))
@@
     (stroke (width 0) (type default))
   )
-  (wire (pts (xy 97.79 186.69) (xy 97.79 187.96))
-    (stroke (width 0) (type default))
-  )
   (wire (pts (xy 233.68 73.025) (xy 233.68 74.295))
     (stroke (width 0) (type default))
@@
     (stroke (width 0) (type default))
   )
-  (wire (pts (xy 100.33 196.85) (xy 100.33 198.12))
-    (stroke (width 0) (type default))
-  )
   (wire (pts (xy 113.03 173.99) (xy 174.625 173.99))
     (stroke (width 0) (type default))
@@
     (stroke (width 0) (type default))
   )
-  (wire (pts (xy 97.79 196.85) (xy 100.33 196.85))
-    (stroke (width 0) (type default))
-  )
   (polyline (pts (xy 368.3 41.91) (xy 368.3 90.805))
     (stroke (width 0) (type default))
@@
     (stroke (width 0) (type default))
   )
-  (wire (pts (xy 97.79 195.58) (xy 97.79 196.85))
-    (stroke (width 0) (type default))
-  )
   (wire (pts (xy 146.05 148.59) (xy 146.05 153.67))
     (stroke (width 0) (type default))
@@
   )
   (wire (pts (xy 150.495 99.06) (xy 166.37 99.06))
-    (stroke (width 0) (type default))
-  )
-  (wire (pts (xy 100.33 186.69) (xy 100.33 196.85))
     (stroke (width 0) (type default))
   )
@@
     (effects (font (size 2.54 2.54) (thickness 0.508) bold) (justify left bottom))
   )
-  (text "JTAG" (at 76.2 169.545 0)
-    (effects (font (size 2.54 2.54) (thickness 0.508) bold) (justify left bottom))
-  )
   (text "UART DEBUG" (at 328.93 142.24 0)
     (effects (font (size 2.54 2.54) (thickness 0.508) bold) (justify left bottom))
@@
     )
   )
-  (symbol (lib_id "Resistor_JLC:0") (at 100.33 152.4 0) (unit 1)
-    (in_bom yes) (on_board yes) (dnp no) (fields_autoplaced)
-    (property "Reference" "R11" (at 102.108 151.7563 0)
-      (effects (font (size 1.27 1.27)) (justify left))
-    )
-    (property "Value" "0" (at 102.108 153.6773 0)
-      (effects (font (size 1.27 1.27)) (justify left))
-    )
-    (property "Footprint" "Resistor_SMD:R_0805_2012Metric_Pad1.20x1.40mm_HandSolder" (at 98.552 152.4 90)
-      (effects (font (size 1.27 1.27)) hide)
-    )
-    (property "Datasheet" "~" (at 100.33 152.4 0)
-      (effects (font (size 1.27 1.27)) hide)
-    )
-    (property "LCSC" "C17477" (at 100.33 152.4 0)
-      (effects (font (size 1.27 1.27)) hide)
-    )
-    (pin "1")
-    (pin "2")
-    (instances
-      (project "Spark-Analyzer"
-        (path "/e63e39d7-6ac0-4ffd-8aa3-1841a4541b55/dc0e84e0-adcd-432b-9bb1-644eba2790b5"
-          (reference "R11") (unit 1)
-        )
-      )
-    )
-  )
   (symbol (lib_id "Resistor_JLC:2.7k") (at 358.14 204.47 0) (unit 1)
     (in_bom yes) (on_board yes) (dnp no) (fields_autoplaced)
@@
         (path "/e63e39d7-6ac0-4ffd-8aa3-1841a4541b55/dc0e84e0-adcd-432b-9bb1-644eba2790b5"
           (reference "R22") (unit 1)
-        )
-      )
-    )
-  )
-  (symbol (lib_id "Resistor_JLC:0") (at 97.79 191.77 0) (unit 1)
-    (in_bom yes) (on_board yes) (dnp no)
-    (property "Reference" "R9" (at 96.012 191.1263 0)
-      (effects (font (size 1.27 1.27)) (justify right))
-    )
-    (property "Value" "0" (at 96.012 193.0473 0)
-      (effects (font (size 1.27 1.27)) (justify right))
-    )
-    (property "Footprint" "Resistor_SMD:R_0805_2012Metric_Pad1.20x1.40mm_HandSolder" (at 96.012 191.77 90)
-      (effects (font (size 1.27 1.27)) hide)
-    )
-    (property "Datasheet" "~" (at 97.79 191.77 0)
-      (effects (font (size 1.27 1.27)) hide)
-    )
-    (property "LCSC" "C17477" (at 97.79 191.77 0)
-      (effects (font (size 1.27 1.27)) hide)
-    )
-    (pin "1")
-    (pin "2")
-    (instances
-      (project "Spark-Analyzer"
-        (path "/e63e39d7-6ac0-4ffd-8aa3-1841a4541b55/dc0e84e0-adcd-432b-9bb1-644eba2790b5"
-          (reference "R9") (unit 1)
         )
       )
@@
         (path "/e63e39d7-6ac0-4ffd-8aa3-1841a4541b55/dc0e84e0-adcd-432b-9bb1-644eba2790b5"
           (reference "#PWR033") (unit 1)
-        )
-      )
-    )
-  )
-  (symbol (lib_id "power:GND") (at 100.33 198.12 0) (unit 1)
-    (in_bom yes) (on_board yes) (dnp no) (fields_autoplaced)
-    (property "Reference" "#PWR017" (at 100.33 204.47 0)
-      (effects (font (size 1.27 1.27)) hide)
-    )
-    (property "Value" "GND" (at 100.33 202.2555 0)
-      (effects (font (size 1.27 1.27)))
-    )
-    (property "Footprint" "" (at 100.33 198.12 0)
-      (effects (font (size 1.27 1.27)) hide)
-    )
-    (property "Datasheet" "" (at 100.33 198.12 0)
-      (effects (font (size 1.27 1.27)) hide)
-    )
-    (pin "1")
-    (instances
-      (project "Spark-Analyzer"
-        (path "/e63e39d7-6ac0-4ffd-8aa3-1841a4541b55/dc0e84e0-adcd-432b-9bb1-644eba2790b5"
-          (reference "#PWR017") (unit 1)
         )
       )
@@
         (path "/e63e39d7-6ac0-4ffd-8aa3-1841a4541b55/dc0e84e0-adcd-432b-9bb1-644eba2790b5"
           (reference "#PWR035") (unit 1)
-        )
-      )
-    )
-  )
-  (symbol (lib_id "power:+3V3") (at 100.33 148.59 0) (unit 1)
-    (in_bom yes) (on_board yes) (dnp no)
-    (property "Reference" "#PWR015" (at 100.33 152.4 0)
-      (effects (font (size 1.27 1.27)) hide)
-    )
-    (property "Value" "+3V3" (at 100.33 145.0881 0)
-      (effects (font (size 1.27 1.27)))
-    )
-    (property "Footprint" "" (at 100.33 148.59 0)
-      (effects (font (size 1.27 1.27)) hide)
-    )
-    (property "Datasheet" "" (at 100.33 148.59 0)
-      (effects (font (size 1.27 1.27)) hide)
-    )
-    (pin "1")
-    (instances
-      (project "Spark-Analyzer"
-        (path "/e63e39d7-6ac0-4ffd-8aa3-1841a4541b55/dc0e84e0-adcd-432b-9bb1-644eba2790b5"
-          (reference "#PWR015") (unit 1)
         )
       )
@@
         )
       )
-    )
-  )
-  (symbol (lib_id "personal:TC2050-IDC") (at 116.84 148.59 0) (unit 1)
-    (in_bom yes) (on_board yes) (dnp no) (fields_autoplaced)
-    (property "Reference" "J2" (at 102.2859 155.7401 0)
-      (effects (font (size 1.27 1.27)) (justify left))
-    )
-    (property "Value" "TC2050-IDC" (at 102.2859 157.6611 0)
-      (effects (font (size 1.27 1.27)) (justify left))
-    )
-    (property "Footprint" "TC2050-IDC" (at 135.89 146.05 0)
-      (effects (font (size 1.27 1.27)) (justify left) hide)
-    )
-    (property "Datasheet" "https://datasheet.datasheetarchive.com/originals/distributors/Datasheets_SAMA/51f607a36a24a0aceedaa5d6ebc30014.pdf" (at 135.89 148.59 0)
-      (effects (font (size 1.27 1.27)) (justify left) hide)
-    )
-    (property "Description" "Plug of nails cable" (at 135.89 151.13 0)
-      (effects (font (size 1.27 1.27)) (justify left) hide)
-    )
-    (property "Manufacturer_Name" "Tag Connect" (at 135.89 156.21 0)
-      (effects (font (size 1.27 1.27)) (justify left) hide)
-    )
-    (property "Manufacturer_Part_Number" "TC2050-IDC" (at 135.89 158.75 0)
-      (effects (font (size 1.27 1.27)) (justify left) hide)
-    )
-    (pin "1")
-    (pin "10")
-    (pin "2")
-    (pin "3")
-    (pin "4")
-    (pin "5")
-    (pin "6")
-    (pin "7")
-    (pin "7")
-    (pin "8")
-    (pin "9")
-    (instances
-      (project "Spark-Analyzer"
-        (path "/e63e39d7-6ac0-4ffd-8aa3-1841a4541b55/dc0e84e0-adcd-432b-9bb1-644eba2790b5"
-          (reference "J2") (unit 1)
-        )
-      )

Commit message: To be reviewed
Parts:
- renumbered R16 to R18, R16 to R22
