File: pcb/Spark-Analyzer/power.kicad_sch (KiCad schematic)
At the start: 20 parts, among them IC4 TPS62175DQCT

Commit message: To be reviewed
Parts:
- renumbered TP5 to TP10, TP5 to TP11, TP5 to TP3, TP5 to TP4
